File: Hardware/MSP430FR4133_DevBoard/DevBoard.brd (EAGLE design)
At the start: 39.5 x 52 mm, 29 parts, among them IC1 TLV75801PDRVT, U1 MSP430FR4133IG56R, Y1 ABS05-32.768KHZ-9-T

Commit message: hardware updates
Parts:
- R4: value (none) -> 5K
- R5: value (none) -> 1K
- U1: value MSP430FR4133IG56R -> MSP430FR4133IG56RDGG56-CLEAN; device MSP430FR4133IG56R:DGG56 -> MSP430FR4133IG56R:DGG56_CLEAN
Routing:
- net GND: vias 5 -> 7
- added copper zone on layer 1, net GND
- added copper zone on layer 16, net GND
Changed lines of the file:
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@@
 <?xml version="1.0" encoding="utf-8"?>
 <!DOCTYPE eagle SYSTEM "eagle.dtd">
-<eagle version="9.3.1">
+<eagle version="9.3.2">
 <drawing>
 <settings>
@@
 <param name="mdViaViaSameLayer" value="6mil"/>
 <param name="mnLayersViaInSmd" value="2"/>
-<param name="mdCopperDimension" value="40mil"/>
+<param name="mdCopperDimension" value="0mil"/>
 <param name="mdDrill" value="6mil"/>
 <param name="mdSmdStop" value="0mil"/>
@@
 <attribute name="VALUE" x="28.231" y="8.085" size="1.27" layer="27" rot="R270"/>
 </element>
-<element name="R4" library="rcl" library_urn="urn:adsk.eagle:library:334" package="R0805" package3d_urn="urn:adsk.eagle:package:23553/2" value="" x="15.06" y="41.04" smashed="yes" rot="R270">
+<element name="R4" library="rcl" library_urn="urn:adsk.eagle:library:334" package="R0805" package3d_urn="urn:adsk.eagle:package:23553/2" value="5K" x="15.06" y="41.04" smashed="yes" rot="R270">
 <attribute name="NAME" x="16.33" y="41.675" size="1.27" layer="25" rot="R270"/>
 <attribute name="SPICEPREFIX" value="R" x="-53.52" y="10.56" size="1.778" layer="27" rot="R270" display="off"/>
 <attribute name="VALUE" x="12.52" y="41.675" size="1.27" layer="27" rot="R270"/>
 </element>
-<element name="R5" library="rcl" library_urn="urn:adsk.eagle:library:334" package="R0805" package3d_urn="urn:adsk.eagle:package:23553/2" value="" x="15.86" y="43.65" smashed="yes" rot="R180">
+<element name="R5" library="rcl" library_urn="urn:adsk.eagle:library:334" package="R0805" package3d_urn="urn:adsk.eagle:package:23553/2" value="1K" x="15.86" y="43.65" smashed="yes" rot="R180">
 <attribute name="NAME" x="16.495" y="42.38" size="1.27" layer="25" rot="R180"/>
 <attribute name="SPICEPREFIX" value="R" x="-19.7" y="112.23" size="1.778" layer="27" rot="R180" display="off"/>
@@
 <attribute name="VALUE" x="8.91" y="13.161" size="1.27" layer="27" align="center"/>
 </element>
-<element name="U1" library="MSP430FR4133IG56R" package="DGG56" value="MSP430FR4133IG56R" x="19.57" y="28.26" smashed="yes">
-<attribute name="MANUFACTURER_PART_NUMBER" value="MSP430FR4133IG56R" x="46.24" y="7.94" size="1.778" layer="27" display="off"/>
+<element name="U1" library="MSP430FR4133IG56R" package="DGG56_CLEAN" value="MSP430FR4133IG56RDGG56-CLEAN" x="19.57" y="28.26" smashed="yes">
 <attribute name="NAME" x="16.2934" y="27.625" size="1.27" layer="25" ratio="6" rot="SR0"/>
-<attribute name="VENDOR" value="Texas Instruments" x="46.24" y="7.94" size="1.778" layer="27" display="off"/>
 </element>
 <element name="Y1" library="ABS05-32.768KHZ-9-T" package="ABS05" value="ABS05-32.768KHZ-9-T" x="10.64" y="29.58" smashed="yes" rot="R90">
@@
 <wire x1="30.771" y1="11.91" x2="30.771" y2="12.269" width="0.4064" layer="1"/>
 <wire x1="30.771" y1="12.269" x2="27.93" y2="15.11" width="0.4064" layer="1"/>
+<polygon width="0.254" layer="1" isolate="0.254">
+<vertex x="0.04" y="52.01"/>
+<vertex x="39.5" y="52.01"/>
+<vertex x="39.5" y="0.02"/>
+<vertex x="0.04" y="0.02"/>
+</polygon>
+<polygon width="0.254" layer="16" isolate="0.254">
+<vertex x="0.04" y="52.01"/>
+<vertex x="39.5" y="52.01"/>
+<vertex x="39.5" y="0.02"/>
+<vertex x="0.04" y="0.02"/>
+</polygon>
+<via x="23.08" y="46.19" extent="1-16" drill="0.508"/>
+<via x="18.46" y="25.23" extent="1-16" drill="0.508"/>
 </signal>
 <signal name="+3V3">
