File: Hardware/MSP430FR4133_DevBoard/DevBoard.sch (EAGLE design)
At the start: 26 parts, among them IC1 TLV75801PDRVT, U1 MSP430FR4133IG56R, Y1 ABS05-32.768KHZ-9-T

Commit message: hardware updates
Parts:
- R4: value (none) -> 5K
- R5: value (none) -> 1K
- U1: value MSP430FR4133IG56R -> MSP430FR4133IG56RDGG56-CLEAN; device MSP430FR4133IG56R:MSP430FR4133IG56R -> MSP430FR4133IG56R:MSP430FR4133IG56RDGG56-CLEAN
Changed lines of the file:
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@@
 <?xml version="1.0" encoding="utf-8"?>
 <!DOCTYPE eagle SYSTEM "eagle.dtd">
-<eagle version="9.3.1">
+<eagle version="9.3.2">
 <drawing>
 <settings>
@@
 <part name="GND5" library="supply1" library_urn="urn:adsk.eagle:library:371" deviceset="GND" device=""/>
 <part name="+3V2" library="supply1" library_urn="urn:adsk.eagle:library:371" deviceset="+3V3" device=""/>
-<part name="U1" library="MSP430FR4133IG56R" deviceset="MSP430FR4133IG56R" device=""/>
+<part name="U1" library="MSP430FR4133IG56R" deviceset="MSP430FR4133IG56R" device="DGG56-CLEAN" value="MSP430FR4133IG56RDGG56-CLEAN"/>
 <part name="Y1" library="ABS05-32.768KHZ-9-T" deviceset="ABS05-32.768KHZ-9-T" device=""/>
 <part name="C7" library="rcl" library_urn="urn:adsk.eagle:library:334" deviceset="C-EU" device="C0805K" package3d_urn="urn:adsk.eagle:package:23681/2"/>
@@
 <part name="C1" library="rcl" library_urn="urn:adsk.eagle:library:334" deviceset="C-EU" device="C0805K" package3d_urn="urn:adsk.eagle:package:23681/2"/>
 <part name="C2" library="rcl" library_urn="urn:adsk.eagle:library:334" deviceset="C-EU" device="C0805K" package3d_urn="urn:adsk.eagle:package:23681/2"/>
-<part name="R4" library="rcl" library_urn="urn:adsk.eagle:library:334" deviceset="R-EU_" device="R0805" package3d_urn="urn:adsk.eagle:package:23553/2"/>
-<part name="R5" library="rcl" library_urn="urn:adsk.eagle:library:334" deviceset="R-EU_" device="R0805" package3d_urn="urn:adsk.eagle:package:23553/2"/>
+<part name="R4" library="rcl" library_urn="urn:adsk.eagle:library:334" deviceset="R-EU_" device="R0805" package3d_urn="urn:adsk.eagle:package:23553/2" value="5K"/>
+<part name="R5" library="rcl" library_urn="urn:adsk.eagle:library:334" deviceset="R-EU_" device="R0805" package3d_urn="urn:adsk.eagle:package:23553/2" value="1K"/>
 <part name="P+3" library="supply1" library_urn="urn:adsk.eagle:library:371" deviceset="+5V" device=""/>
 <part name="+3V4" library="supply1" library_urn="urn:adsk.eagle:library:371" deviceset="+3V3" device=""/>
